File: PicoAlt.kicad_sch (KiCad schematic)
At the start: 35 parts, among them J2 USB_B, J3 Conn_01x04, J4 Conn_01x20, J5 Conn_01x20, SW1 SW_Push, U1 AMS1117-3.3, U2 W25Q128JVSIQ, U3 RP2040, Y1 12 MHz

Commit message: JLCPCB submit
Parts:
- removed JP2: PROG, Connector_PinHeader_2.54mm:PinHeader_1x02_P2.54mm_Vertical, symbol Jumper:Jumper_2_Open
- added D1: LED, LED_SMD:LED_0603_1608Metric_Pad1.05x0.95mm_HandSolder, symbol Device:LED
- added R1: 1k, Resistor_SMD:R_0603_1608Metric_Pad0.98x0.95mm_HandSolder, symbol Device:R
- added SW2: SW_Push, PicoAlt:K2-1808UN, symbol Switch:SW_Push
- SW1: footprint Button_Switch_THT:SW_PUSH_6mm -> PicoAlt:K2-1808UN; LCSC (none) -> C145878
Connections:
- net GND: now also D1.1 (K), SW2.2
- net GPIO25: now also R1.2
- net at R9.2: now also SW2.1
- new net: D1.2 (A), R1.1
Other:
- note added: "https://jlcpcb.com/partdetail/157210-K2_1808UN_A4SW04/C145878"
Changed lines of the file:
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@@
+    (stroke (width 0) (type default) (color 0 0 0 0))
+  )
+  (wire (pts (xy 208.915 123.825) (xy 208.915 125.095))
     (stroke (width 0) (type default) (color 0 0 0 0))
   )
@@
     (stroke (width 0) (type default) (color 0 0 0 0))
   )
+  (text "https://jlcpcb.com/partdetail/157210-K2_1808UN_A4SW04/C145878"
+    (at 192.405 150.495 0)
+    (effects (font (size 1.27 1.27)) (justify left bottom))
+  )
   (global_label "GPIO16" (shape input) (at 245.11 103.505 0) (fields_autoplaced)
     (effects (font (size 1.27 1.27)) (justify left))
@@
     (property "Intersheet References" "${INTERSHEET_REFS}" (id 0) (at 197.7026 90.0906 0)
       (effects (font (size 1.27 1.27)) (justify right) hide)
+    )
+  )
+  (global_label "GPIO25" (shape input) (at 208.915 123.825 90) (fields_autoplaced)
+    (effects (font (size 1.27 1.27)) (justify left))
+    (property "Intersheet References" "${INTERSHEET_REFS}" (id 0) (at 208.8356 114.5176 90)
+      (effects (font (size 1.27 1.27)) (justify left) hide)
     )
   )
@@
     (pin "1")
   )
+  (symbol (lib_id "Device:LED") (at 208.915 136.525 90) (unit 1)
+    (in_bom yes) (on_board yes) (fields_autoplaced)
+    (property "Reference" "D1" (id 0) (at 212.09 136.8424 90)
+      (effects (font (size 1.27 1.27)) (justify right))
+    )
+    (property "Value" "LED" (id 1) (at 212.09 139.3824 90)
+      (effects (font (size 1.27 1.27)) (justify right))
+    )
+    (property "Footprint" "LED_SMD:LED_0603_1608Metric_Pad1.05x0.95mm_HandSolder" (id 2) (at 208.915 136.525 0)
+      (effects (font (size 1.27 1.27)) hide)
+    )
+    (property "Datasheet" "~" (id 3) (at 208.915 136.525 0)
+      (effects (font (size 1.27 1.27)) hide)
+    )
+    (property "LCSC" "C2286" (id 4) (at 208.915 136.525 90)
+      (effects (font (size 1.27 1.27)) hide)
+    )
+    (pin "1")
+    (pin "2")
+  )
   (symbol (lib_id "power:GND") (at 146.685 41.275 0) (unit 1)
     (in_bom yes) (on_board yes) (fields_autoplaced)
@@
     )
     (pin "1")
+  )
+  (symbol (lib_id "Switch:SW_Push") (at 62.23 156.845 0) (unit 1)
+    (in_bom yes) (on_board yes) (fields_autoplaced)
+    (property "Reference" "SW2" (id 0) (at 62.23 149.225 0))
+    (property "Value" "SW_Push" (id 1) (at 62.23 151.765 0))
+    (property "Footprint" "PicoAlt:K2-1808UN" (id 2) (at 62.23 151.765 0)
+      (effects (font (size 1.27 1.27)) hide)
+    )
+    (property "Datasheet" "~" (id 3) (at 62.23 151.765 0)
+      (effects (font (size 1.27 1.27)) hide)
+    )
+    (property "LCSC" "C145878" (id 4) (at 62.23 156.845 0)
+      (effects (font (size 1.27 1.27)) hide)
+    )
+    (pin "1")
+    (pin "2")
   )
   (symbol (lib_id "PicoAlt:SOIC8Flash") (at 68.58 178.435 0) (unit 1)
@@
     (property "Reference" "SW1" (id 0) (at 86.36 114.3 0))
     (property "Value" "SW_Push" (id 1) (at 86.36 116.84 0))
-    (property "Footprint" "Button_Switch_THT:SW_PUSH_6mm" (id 2) (at 86.36 116.84 0)
+    (property "Footprint" "PicoAlt:K2-1808UN" (id 2) (at 86.36 116.84 0)
       (effects (font (size 1.27 1.27)) hide)
     )
     (property "Datasheet" "~" (id 3) (at 86.36 116.84 0)
+      (effects (font (size 1.27 1.27)) hide)
+    )
+    (property "LCSC" "C145878" (id 4) (at 86.36 121.92 0)
       (effects (font (size 1.27 1.27)) hide)
     )
@@
     )
     (pin "1")
+  )
+  (symbol (lib_id "Device:R") (at 208.915 128.905 180) (unit 1)
+    (in_bom yes) (on_board yes)
+    (property "Reference" "R1" (id 0) (at 211.455 128.905 90))
+    (property "Value" "1k" (id 1) (at 208.915 128.905 90))
+    (property "Footprint" "Resistor_SMD:R_0603_1608Metric_Pad0.98x0.95mm_HandSolder" (id 2) (at 210.693 128.905 90)
+      (effects (font (size 1.27 1.27)) hide)
+    )
+    (property "Datasheet" "~" (id 3) (at 208.915 128.905 0)
+      (effects (font (size 1.27 1.27)) hide)
+    )
+    (property "LCSC" "C21190" (id 4) (at 208.915 128.905 90)
+      (effects (font (size 1.27 1.27)) hide)
+    )
+    (pin "1")
+    (pin "2")
   )
   (symbol (lib_id "Connector_Generic:Conn_01x20") (at 233.68 80.645 180) (unit 1)
@@
     (pin "1")
   )
+  (symbol (lib_id "power:GND") (at 208.915 140.335 0) (unit 1)
+    (in_bom yes) (on_board yes) (fields_autoplaced)
+    (property "Reference" "#PWR0120" (id 0) (at 208.915 146.685 0)
+      (effects (font (size 1.27 1.27)) hide)
+    )
+    (property "Value" "GND" (id 1) (at 208.915 144.78 0))
+    (property "Footprint" "" (id 2) (at 208.915 140.335 0)
+      (effects (font (size 1.27 1.27)) hide)
+    )
+    (property "Datasheet" "" (id 3) (at 208.915 140.335 0)
+      (effects (font (size 1.27 1.27)) hide)
+    )
+    (pin "1")
+  )
   (symbol (lib_id "Regulator_Linear:AMS1117-3.3") (at 34.925 94.615 0) (unit 1)
     (in_bom yes) (on_board yes) (fields_autoplaced)
@@
     )
     (property "LCSC" "C1555" (id 4) (at 90.17 109.22 0)
-      (effects (font (size 1.27 1.27)) hide)
-    )
-    (pin "1")
-    (pin "2")
-  )
-  (symbol (lib_id "Jumper:Jumper_2_Open") (at 62.23 156.845 0) (unit 1)
-    (in_bom yes) (on_board yes) (fields_autoplaced)
-    (property "Reference" "JP2" (id 0) (at 62.23 149.86 0))
-    (property "Value" "PROG" (id 1) (at 62.23 152.4 0))
-    (property "Footprint" "Connector_PinHeader_2.54mm:PinHeader_1x02_P2.54mm_Vertical" (id 2) (at 62.23 156.845 0)
-      (effects (font (size 1.27 1.27)) hide)
-    )
-    (property "Datasheet" "~" (id 3) (at 62.23 156.845 0)
       (effects (font (size 1.27 1.27)) hide)
     )
@@
       (reference "#PWR0119") (unit 1) (value "GND") (footprint "")
     )
+    (path "/a975845b-c88e-47dc-9b6e-26265bcea023"
+      (reference "#PWR0120") (unit 1) (value "GND") (footprint "")
+    )
     (path "/240858a0-7b8e-4b5d-95bf-5de9673b377e"
       (reference "#PWR0121") (unit 1) (value "GND") (footprint "")
@@
       (reference "C18") (unit 1) (value "2.2 uF") (footprint "Capacitor_SMD:C_0603_1608Metric")
     )
+    (path "/39dd035f-0f97-493f-924b-700658a8bbb3"
+      (reference "D1") (unit 1) (value "LED") (footprint "LED_SMD:LED_0603_1608Metric_Pad1.05x0.95mm_HandSolder")
+    )
     (path "/056181b2-6ba5-4fa9-84cd-e737be9981d5"
       (reference "D2") (unit 1) (value "SS14") (footprint "Diode_SMD:D_SMA")
@@
       (reference "JP1") (unit 1) (value "ADC3") (footprint "Connector_PinHeader_2.54mm:PinHeader_1x02_P2.54mm_Vertical")
     )
-    (path "/d1258ea5-6259-4354-869f-0c70820b98e4"
-      (reference "JP2") (unit 1) (value "PROG") (footprint "Connector_PinHeader_2.54mm:PinHeader_1x02_P2.54mm_Vertical")
+    (path "/91360d2d-cc65-4a74-a608-518ef882cb51"
+      (reference "R1") (unit 1) (value "1k") (footprint "Resistor_SMD:R_0603_1608Metric_Pad0.98x0.95mm_HandSolder")
     )
     (path "/9b501e98-6f36-4c2f-b90f-d46fe5842bff"
@@
     )
     (path "/80adae98-f4cb-4d1e-b25d-50e1f734760b"
-      (reference "SW1") (unit 1) (value "SW_Push") (footprint "Button_Switch_THT:SW_PUSH_6mm")
+      (reference "SW1") (unit 1) (value "SW_Push") (footprint "PicoAlt:K2-1808UN")
+    )
+    (path "/6a2c007c-6d60-4d2f-9aaa-2e35a2aa628d"
+      (reference "SW2") (unit 1) (value "SW_Push") (footprint "PicoAlt:K2-1808UN")
     )
     (path "/aac4f9d6-7597-44c3-9dfe-d5677b0543d4"

Commit message: Modified for bigger SOIC-8 footprint
Parts:
- U2: footprint Package_SO:SOIC-8_3.9x4.9mm_P1.27mm -> PicoAlt:SOIC-8_3.9x4.9mm_P1.27mm_mod
Changed lines of the file:
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@@
     (property "Reference" "U2" (id 0) (at 67.6275 167.64 0))
     (property "Value" "W25Q128JVSIQ" (id 1) (at 67.6275 170.18 0))
-    (property "Footprint" "Package_SO:SOIC-8_3.9x4.9mm_P1.27mm" (id 2) (at 62.865 179.07 0)
+    (property "Footprint" "PicoAlt:SOIC-8_3.9x4.9mm_P1.27mm_mod" (id 2) (at 62.865 179.07 0)
       (effects (font (size 1.27 1.27)) hide)
     )
@@
     )
     (path "/6b259622-36c2-4bda-9154-14bc2de13062"
-      (reference "U2") (unit 1) (value "W25Q128JVSIQ") (footprint "Package_SO:SOIC-8_3.9x4.9mm_P1.27mm")
+      (reference "U2") (unit 1) (value "W25Q128JVSIQ") (footprint "PicoAlt:SOIC-8_3.9x4.9mm_P1.27mm_mod")
     )
     (path "/fad21c40-788f-48ce-b290-9d267f63ec0a"
