File: PicoAlt.kicad_pcb (KiCad board)
At the start: 2 copper layers, 20.3 x 57.8 mm, 35 parts, among them J2 USB_B, J3 Conn_01x04, J4 Conn_01x20, J5 Conn_01x20, SW1 SW_Push, U1 AMS1117-3.3, U2 W25Q128JVSIQ, U3 RP2040, Y1 12 MHz

Commit message: JLCPCB submit
Parts:
- removed JP2: PROG, Connector_PinHeader_2.54mm:PinHeader_1x02_P2.54mm_Vertical
- added D1: LED, LED_SMD:LED_0603_1608Metric_Pad1.05x0.95mm_HandSolder, F.Cu at (154.9, 109.0)
- added R1: 1k, Resistor_SMD:R_0603_1608Metric_Pad0.98x0.95mm_HandSolder, F.Cu at (154.8, 105.6)
- added SW2: SW_Push, PicoAlt:K2-1808UN, F.Cu at (144.4, 124.8)
- SW1: footprint Button_Switch_THT:SW_PUSH_6mm -> PicoAlt:K2-1808UN
- moved SW1 2.30 mm to (152.6, 124.8), turned to 90 degrees
- moved R6 1.10 mm to (151.7, 111.7)
- moved C11 0.67 mm to (153.5, 106.0), turned to 90 degrees
- moved R7 0.21 mm to (153.8, 100.2)
- moved C8 0.18 mm to (154.1, 102.5)
Routing:
- net GND: track 44.3 -> 48.5 mm, vias 37 -> 42
- net GPIO25: track 0.00 -> 3.24 mm
- net Net-(R9-Pad2): track 8.98 -> 12.0 mm
- net RUN: track 33.6 -> 30.8 mm
- net +3.3V: track 111.3 -> 109.5 mm
- net Net-(D1-Pad2): track 0.00 -> 1.56 mm
- net GPIO17: track 19.7 -> 18.4 mm
- net GPIO3: track 18.9 -> 20.0 mm
- net GPIO16: track 22.3 -> 21.3 mm
- net GPIO18: track 14.6 -> 13.6 mm
- net Net-(J3-Pad2): track 16.8 -> 15.8 mm
- net GPIO21: track 8.62 -> 9.49 mm
- net Net-(J3-Pad4): track 13.0 -> 12.2 mm
- net GPIO20: track 10.5 -> 11.2 mm
Other:
- board text added: "RESET"
- board text added: "SWCLK"
- board text added: "SWIO"
- board text removed: "CLK"
- board text removed: "SWD"

Commit message: Modified for bigger SOIC-8 footprint
Parts:
- U2: footprint Package_SO:SOIC-8_3.9x4.9mm_P1.27mm -> PicoAlt:SOIC-8_3.9x4.9mm_P1.27mm_mod
- moved U2 0.20 mm to (147.2, 94.7)
Routing:
- net +3.3V: track 109.5 -> 105.1 mm, vias 4 -> 5
- net ADCVREF: track 16.3 -> 14.4 mm, vias 0 -> 1
- net QSPISS: track 25.7 -> 26.9 mm
- net GPIO29: track 12.3 -> 13.1 mm
- net QSPISD0: track 8.25 -> 7.56 mm
- net QSPISD1: track 10.7 -> 11.3 mm
- net QSPICLK: track 11.6 -> 12.1 mm

Commit message: JLCPCB #2
Routing:
- net +1V1: track 16.9 -> 19.9 mm, vias 0 -> 2
- net GND: track 48.5 -> 47.9 mm, vias 42 -> 41
